File: Hermes/Hermes.kicad_pcb (KiCad board)
At the start: 4 copper layers, 39 x 15.5 mm, 38 parts, among them J1 USB_B_Micro, J2 Conn_ARM_JTAG_SWD_10, J3 SMA, U1 XC6206P332MR, U2 USBLC6-2SC6, U3 STM32L432KBU6, U4 nRF24L01P, Y1 16MHz

Commit message: Documentation
Routing:
- net GND: track 89.9 -> 86.8 mm
Changed lines of the file:
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@@
   (segment (start 161.198008 90.1) (end 161.925 89.373008) (width 0.25) (layer "F.Cu") (net 2))
   (segment (start 167.1625 89.54) (end 167.1625 88.5875) (width 0.29337) (layer "F.Cu") (net 2))
-  (segment (start 161.45 84.85) (end 161.45 85.175) (width 0.25) (layer "F.Cu") (net 2))
   (segment (start 163.175 98.325) (end 163.15 98.35) (width 0.8) (layer "F.Cu") (net 2))
   (segment (start 170.775 98.375) (end 171.85 98.375) (width 0.8) (layer "F.Cu") (net 2))
@@
   (segment (start 163.1875 98.25) (end 163.15 98.2875) (width 0.8) (layer "F.Cu") (net 2))
   (segment (start 161.8375 97.925) (end 161.8375 98.3125) (width 0.25) (layer "F.Cu") (net 2))
-  (segment (start 160.7 84.1) (end 161.45 84.85) (width 0.25) (layer "F.Cu") (net 2))
   (segment (start 158.8 93.175) (end 158.8 92.5375) (width 0.25) (layer "F.Cu") (net 2))
   (segment (start 159.3 87.09) (end 159.35 87.04) (width 0.25) (layer "F.Cu") (net 2))
@@
   (segment (start 140.34 95.855) (end 140.34 94.99) (width 0.4) (layer "F.Cu") (net 2))
   (segment (start 152.05 85.1575) (end 153.225 86.3325) (width 0.4) (layer "F.Cu") (net 2))
-  (segment (start 159.15 84.375) (end 159.425 84.1) (width 0.25) (layer "F.Cu") (net 2))
   (segment (start 157.975 94.2) (end 157.105 94.2) (width 0.25) (layer "F.Cu") (net 2))
   (segment (start 161.55875 97.58375) (end 161.8375 97.8625) (width 0.25) (layer "F.Cu") (net 2))
@@
   (segment (start 163.15 98.35) (end 163.175 98.375) (width 0.8) (layer "F.Cu") (net 2))
   (segment (start 144.125 86.65) (end 143.975 86.5) (width 0.8) (layer "F.Cu") (net 2))
-  (segment (start 159.425 84.1) (end 160.7 84.1) (width 0.25) (layer "F.Cu") (net 2))
   (segment (start 161.5875 97.675) (end 161.8375 97.925) (width 0.25) (layer "F.Cu") (net 2))
   (segment (start 147.745 93.705) (end 147.75 93.7) (width 0.25) (layer "F.Cu") (net 2))
