File: Hermes/Hermes.kicad_sch (KiCad schematic)
At the start: 38 parts, among them J1 USB_B_Micro, J2 Conn_ARM_JTAG_SWD_10, J3 SMA, U1 XC6206P332MR, U2 USBLC6-2SC6, U3 STM32L432KBU6, U4 nRF24L01P, Y1 16MHz

Commit message: Updating schematic comments
Other:
- note added: "+ / - is for the differential pairs. Impedance included in MCU drivers (i.e. no termination R needed)."
- note added: "Ferrite bead to reduce ringing. Fuse (Relatively large footprint for easy replacement) for overload protection."
- note added: "For programming and debugging the STM."
- note added: "Indicator LEDs. Red for TX, yellow for RX."
- note added: "NOTE: For RF impedance matching, we need 50 Ohm traces. Using the stackup information, this means 11.55 mil width traces. For the USB differential signals, we need 90 Ohm differential traces with. Assuming 8mil spacing and stackup, the trace widths should be 10.28 mils."
- note added: "Passive Antenna Setup (Impedance Matching, Biasing, & SMA Connection)"
- note added: "Route with 50 Ohm impedance traces. Assumes 50 Ohm anetenna."
- note added: "Shield is GND at host as per USB spec."
- note added: "This IC supports differntial antenna, but, for cost and simplicity, this will use a single-ended antenna. The matching network handles this change."
- note added: "Three 100n C (one for each VDD pin). One bulk 1u C in vicinity of IC."
- note removed: "+ / - Is for differential pairs! Impedance included in drivers (no termination res. needed)."
- note removed: "Ferrite bead to reduce ringing."
- note removed: "NOTE: For RF impedance matching, we need 50 Ohm traces. Using the stackup information, this mean 11.55 mil width traces. For the USB differential signals, we need 90 Ohm differential traces with. Assuming 8mil spacing, the trace widths should be 10.28 mils."
- note removed: "One 100n cap. for each VDD pin. One bulk 1u cap. in vicinity."
- note removed: "Passive Antenna w/ Impedance Matching & SMA Connection"
- note removed: "Route with 50 Ohm impedance traces"
- note removed: "Shield is GND at host."
- moved on the sheet: C1, C10, C11, C16, C17, C2, C8, C9, F1, FB1, R5, U1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
